File: Cat_feeder_KiCad/rtc_board.kicad_sch (KiCad schematic)
At the start: 6 parts, among them J3 Conn_01x04_Pin, U5 DS3231M

Commit message: changing schematic bc I was dumb yesterday
Parts:
- C5: footprint (none) -> Capacitor_SMD:C_0805_2012Metric
- J3: footprint (none) -> Connector_PinHeader_2.54mm:PinHeader_1x04_P2.54mm_Horizontal
- R1: footprint (none) -> Resistor_SMD:R_0805_2012Metric
Changed lines of the file:
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@@
 			)
 		)
-		(property "Footprint" ""
+		(property "Footprint" "Resistor_SMD:R_0805_2012Metric"
 			(at 222.25 93.218 90)
 			(hide yes)
@@
 			)
 		)
-		(property "Footprint" ""
+		(property "Footprint" "Connector_PinHeader_2.54mm:PinHeader_1x04_P2.54mm_Horizontal"
 			(at 138.43 91.44 0)
 			(hide yes)
@@
 			)
 		)
-		(property "Footprint" ""
+		(property "Footprint" "Capacitor_SMD:C_0805_2012Metric"
 			(at 209.55 101.9048 0)
 			(hide yes)
