File: Cat_feeder_KiCad/Cat_feeder_KiCad.kicad_sch (KiCad schematic)
At the start: 0 parts

Commit message: doing schematic going okay ig...
Parts:
- added C1, C2, C3: 10uF, Capacitor_SMD:C_0805_2012Metric, symbol Device:C
- added J1: Conn_01x03_Pin, Connector_PinHeader_2.54mm:PinHeader_1x03_P2.54mm_Vertical, symbol Connector:Conn_01x03_Pin
- added R1, R2: 4.7K, Resistor_SMD:R_0805_2012Metric, symbol Device:R
- added R3: 10K, Resistor_SMD:R_0805_2012Metric, symbol Device:R
- added SW1: SW_Push, Button_Switch_THT:SW_PUSH_6mm, symbol Switch:SW_Push
- added U1: ESP32-S3-WROOM-1, RF_Module:ESP32-S3-WROOM-1, symbol RF_Module:ESP32-S3-WROOM-1
- added U2: DS3231M, Package_SO:SOIC-16W_7.5x10.3mm_P1.27mm, symbol Timer_RTC:DS3231M
- added U3: ER_OLEDM0.91_1x-I2C, Display:ER_OLEDM0.91_1x-I2C, symbol Display_Graphic:ER_OLEDM0.91_1x-I2C
- added U4: LD1117V33, Package_TO_SOT_THT:TO-220-3_Vertical, symbol Regulator_Linear:LD1117V33
Connections:
- new net: C1.2, R1.1, R2.1, U1.2 (3V3), U3.2 (VCC), U4.2 (VO)
- new net: SW1.2, U1.21 (IO13)
- new net: J1.3 (Pin_3), U1.10 (IO17)
- new net: R1.2, U1.12 (IO8), U2.15 (SDA)
- new net: R3.2, U1.3 (EN)
- new net: R2.2, U1.17 (IO9), U2.16 (SCL)
- new net +3.3V: U2.2 (VCC)
- new net +3V3: R3.1
- new net +5V: C2.1, J1.2 (Pin_2), U4.3 (VI)
- new net GND: C1.1, C2.2, J1.1 (Pin_1), SW1.1, U1.1 (GND), U1.40 (GND), U1.41 (GND), U2.10 (GND), U2.11 (GND), U2.12 (GND), U2.13 (GND), U2.5 (GND), U2.6 (GND), U2.7 (GND), U2.8 (GND), U2.9 (GND), U3.1 (GND), U4.1 (GND)
- no-connect marks 0 -> 4

Commit message: editing schematic
Parts:
- added BT1: Battery_Cell, symbol Device:Battery_Cell
- added C4, C5: 100nF, Capacitor_SMD:C_0805_2012Metric, symbol Device:C
- added D1: 1N4148, Diode_THT:D_DO-35_SOD27_P7.62mm_Horizontal, symbol Diode:1N4148
- added R4: 10K, Resistor_SMD:R_0805_2012Metric, symbol Device:R
- added SW2: Reset button, symbol Switch:SW_Push
- R3: value 10K -> 100V
Connections:
- net +3.3V: now also R4.2
- net +5V: now also C3.2
- net GND: now also C3.1, BT1.2 (-), C4.2, C5.1, SW2.1, SW2.2
- net at SW1.2, U1.21 (IO13): now also R4.1
- net at U1.3 (EN): now also C4.1; no longer R3.2
- net at U2.14 (VBAT): now also C5.2, D1.1 (K)
- net +3V3: no longer names the net of R3.1
- net +3V3: now also BT1.1 (+)
- new net: D1.2 (A), R3.2
- no-connect marks 4 -> 3
Other:
- moved on the sheet: C3, R3

Commit message: polishing and editing schematic
Parts:
- BT1: footprint (none) -> Battery:BatteryHolder_Keystone_3034_1x20mm
- SW2: footprint (none) -> Button_Switch_THT:SW_PUSH_6mm
Connections:
- net +3.3V: now also C1.2, C4.1, R1.1, R2.1, SW2.2, U1.2 (3V3), U1.3 (EN), U3.2 (VCC), U4.2 (VO)
- net GND: no longer SW2.2
- net at U3.3 (SCL): now also U1.23 (IO21)
- net at U3.4 (SDA): now also U1.31 (IO38)
Other:
- moved on the sheet: BT1, C1, C2, C4, C5, D1, J1, R3, SW2, U3, U4

Commit message: added a sub page onto my schematic
Parts:
- removed BT1: Battery_Cell, Battery:BatteryHolder_Keystone_3034_1x20mm, symbol Device:Battery_Cell
- removed C5: 100nF, Capacitor_SMD:C_0805_2012Metric, symbol Device:C
- removed D1: 1N4148, Diode_THT:D_DO-35_SOD27_P7.62mm_Horizontal, symbol Diode:1N4148
- removed R1, R2: 4.7K, Resistor_SMD:R_0805_2012Metric, symbol Device:R
- removed R3: 100V, Resistor_SMD:R_0805_2012Metric, symbol Device:R
- removed U2: DS3231M, Package_SO:SOIC-16W_7.5x10.3mm_P1.27mm, symbol Timer_RTC:DS3231M
- added J2: Conn_01x04_Pin, symbol Connector:Conn_01x04_Pin
Connections:
- net +3.3V: now also J2.1 (Pin_1)
- net GND: now also J2.2 (Pin_2)
- net SCL_IO18: now reaches U3.3 (SCL)
- net SCL_IO18: now also U1.11 (IO18); no longer U1.23 (IO21)
- net at U1.31 (IO38): no longer U3.4 (SDA)
- net RTC_board/SCL: now reaches U1.18 (IO10)
- net RTC_board/SDA: now reaches U1.19 (IO11)
- new net SCL: J2.4 (Pin_4)
- new net SDA: J2.3 (Pin_3)
- new net SDA_IO21: U1.23 (IO21), U3.4 (SDA)
- no-connect marks 3 -> 0
Other:
- added sheet RTC_board (rtc_board.kicad_sch)

Commit message: changing schematic bc I was dumb yesterday
Parts:
- removed U3: ER_OLEDM0.91_1x-I2C, Display:ER_OLEDM0.91_1x-I2C, symbol Display_Graphic:ER_OLEDM0.91_1x-I2C
- added BT1: Battery_Cell, symbol Device:Battery_Cell
- added C5: 100nF, Capacitor_SMD:C_0805_2012Metric, symbol Device:C
- added D1: 1N4148, Diode_THT:D_DO-35_SOD27_P7.62mm_Horizontal, symbol Diode:1N4148
- added R1: 100Ω, Resistor_SMD:R_0805_2012Metric, symbol Device:R
- added U5: DS3231M, Package_SO:SOIC-16W_7.5x10.3mm_P1.27mm, symbol Timer_RTC:DS3231M
- J2: footprint (none) -> Connector_PinHeader_2.54mm:PinHeader_1x04_P2.54mm_Vertical
Connections:
- net SCL_IO18 is gone; now on net SDA: U1.11 (IO18)
- net SDA_IO21 is gone; now on net SCL: U1.23 (IO21)
- net +3.3V: now also U5.2 (VCC)
- net GND: now also BT1.2 (-), C5.2, U5.10 (GND), U5.11 (GND), U5.12 (GND), U5.13 (GND), U5.5 (GND), U5.6 (GND), U5.7 (GND), U5.8 (GND), U5.9 (GND)
- net SCL: now also J2.3 (Pin_3); no longer J2.4 (Pin_4)
- net SDA: now also J2.4 (Pin_4); no longer J2.3 (Pin_3)
- net SDA_IO: now reaches U1.27 (IO0)
- net SDA_IO: now also U5.15 (SDA)
- net SCL_I0: now reaches U1.39 (IO1)
- net SCL_I0: now also U5.16 (SCL)
- net RTC_board/SCL: no longer names the net of U1.18 (IO10)
- net RTC_board/SDA: no longer names the net of U1.19 (IO11)
- new net: C5.1, D1.1 (K), U5.14 (VBAT)
- new net: D1.2 (A), R1.1
- new net: BT1.1 (+), R1.2
Other:
- removed sheet RTC_board
- moved on the sheet: J2

Commit message: doing schematic
Parts:
- removed BT1: Battery_Cell, symbol Device:Battery_Cell
- removed C5: 100nF, Capacitor_SMD:C_0805_2012Metric, symbol Device:C
- removed D1: 1N4148, Diode_THT:D_DO-35_SOD27_P7.62mm_Horizontal, symbol Diode:1N4148
- removed R1: 100Ω, Resistor_SMD:R_0805_2012Metric, symbol Device:R
- removed U5: DS3231M, Package_SO:SOIC-16W_7.5x10.3mm_P1.27mm, symbol Timer_RTC:DS3231M
- added BT2: Battery_Cell, symbol Device:Battery_Cell
- added C7: 100nF, Capacitor_SMD:C_0805_2012Metric, symbol Device:C
- added C8: 1uF, Capacitor_SMD:C_0805_2012Metric, symbol Device:C
- added D2: 1N4148, Diode_THT:D_DO-35_SOD27_P7.62mm_Horizontal, symbol Diode:1N4148
- added R5: 100Ω, Resistor_SMD:R_0805_2012Metric, symbol Device:R
- added R6, R7, R8: 4.7K, symbol Device:R
- added U5: PCF85263AT, Package_SO:SOIC-8_3.9x4.9mm_P1.27mm, symbol Timer_RTC:PCF85263AT
- added Y1: Crystal, symbol Device:Crystal
Connections:
- net +3.3V: now also C8.2, R6.2, R7.2, R8.2, U5.8 (VDD)
- net GND: now also BT2.2 (-), C7.2, C8.1, U5.4 (VSS)
- net SCL_I0: now also R6.1, U5.6 (SCL)
- net SDA_IO: now also R7.1, U5.5 (SDA)
- net INTA_IO6: now reaches U1.6 (IO6)
- net INTA_IO6: now also R8.1, U5.7 (~{INTA})
- new net: C7.1, D2.1 (K), U5.3 (VBAT)
- new net: D2.2 (A), R5.1
- new net: U5.2 (OSCO), Y1.1
- new net: U5.1 (OSCI), Y1.2
- new net: BT2.1 (+), R5.2
Other:
- moved on the sheet: C1, C2, C3, C4, J1, J2, R4, SW1, SW2, U1, U4

Commit message: adding footprints
Parts:
- BT2: footprint (none) -> Battery:BatteryHolder_Keystone_3034_1x20mm
- R6, R7, R8: footprint (none) -> Resistor_SMD:R_0805_2012Metric
- Y1: footprint (none) -> Crystal:Crystal_SMD_3225-4Pin_3.2x2.5mm
Changed lines of the file:
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@@
 			)
 		)
-		(property "Footprint" ""
+		(property "Footprint" "Resistor_SMD:R_0805_2012Metric"
 			(at 26.162 180.34 90)
 			(hide yes)
@@
 			)
 		)
-		(property "Footprint" ""
+		(property "Footprint" "Crystal:Crystal_SMD_3225-4Pin_3.2x2.5mm"
 			(at 44.45 172.72 0)
 			(hide yes)
@@
 			)
 		)
-		(property "Footprint" ""
+		(property "Footprint" "Resistor_SMD:R_0805_2012Metric"
 			(at 132.588 171.45 90)
 			(hide yes)
@@
 			)
 		)
-		(property "Footprint" ""
+		(property "Footprint" "Battery:BatteryHolder_Keystone_3034_1x20mm"
 			(at 128.27 143.256 90)
 			(hide yes)
@@
 			)
 		)
-		(property "Footprint" ""
+		(property "Footprint" "Resistor_SMD:R_0805_2012Metric"
 			(at 38.862 180.34 90)
 			(hide yes)

Commit message: some schematic work + kicad crashed
Parts:
- Y1: footprint Crystal:Crystal_SMD_3225-4Pin_3.2x2.5mm -> Crystal:Crystal_SMD_0603-2Pin_6.0x3.5mm
Changed lines of the file:
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@@
 			)
 		)
-		(property "Footprint" "Crystal:Crystal_SMD_3225-4Pin_3.2x2.5mm"
+		(property "Footprint" "Crystal:Crystal_SMD_0603-2Pin_6.0x3.5mm"
 			(at 44.45 172.72 0)
 			(hide yes)
