File: Cat_feeder_KiCad/Cat_feeder_KiCad.kicad_sch (KiCad schematic)
At the start: 21 parts, among them J1 Conn_01x03_Pin, J2 Conn_01x04_Pin, SW1 SW_Push, SW2 Reset button, U1 ESP32-S3-WROOM-1, U4 LD1117V33, U5 PCF85263AT, Y1 Crystal

Commit message: deleted a button
Parts:
- removed R4: 10K, Resistor_SMD:R_0805_2012Metric, symbol Device:R
- removed SW1: SW_Push, Button_Switch_THT:SW_PUSH_6mm, symbol Switch:SW_Push
- added J3: USB_C_Receptacle_USB2.0_14P, Connector_USB:USB_C_Receptacle_HRO_TYPE-C-31-M-12, symbol Connector:USB_C_Receptacle_USB2.0_14P
- J1: value Conn_01x03_Pin -> Servo motor connector
- J2: value Conn_01x04_Pin -> OLED connector
Connections:
- net +5V: now also J3.A4 (VBUS), J3.A9 (VBUS), J3.B4 (VBUS), J3.B9 (VBUS)
- net GND: now also J3.A1 (GND), J3.A12 (GND), J3.B1 (GND), J3.B12 (GND)
- net at U1.13 (USB_D-): now also J3.B7 (D-)
- net at U1.14 (USB_D+): now also J3.B6 (D+)
- no-connect marks 0 -> 4
